File: CNC_IO_Buffer_Cape.brd (EAGLE design)
At the start: 79.8 x 80 mm, 172 parts, among them CN1 1X4-CLEANBIG

Commit message: work in progress
Parts:
- moved R21 5.84 mm to (22.9, 55.4), turned to 0 degrees
- moved R23 5.84 mm to (22.9, 50.3), turned to 0 degrees
- moved R35 5.84 mm to (22.9, 45.2), turned to 0 degrees
- moved R37 5.84 mm to (22.9, 40.1), turned to 0 degrees
- moved R43 2.34 mm to (22.9, 35.1)
- moved R13 2.29 mm to (57.1, 8.89), turned to 180 degrees
- moved R19 1.80 mm to (5.59, 31.2)
- moved R1 1.65 mm to (65.7, 27.1)
- moved C1 0.51 mm to (13.7, 5.33)
- moved C19 0.51 mm to (4.45, 23.9)
- moved C2 0.51 mm to (25.1, 5.33)
- moved C3 0.51 mm to (36.6, 5.33)
- moved C4 0.51 mm to (48.0, 5.33)
- moved C5 0.51 mm to (59.4, 5.33)
- moved R38 0.46 mm to (4.70, 19.8), flipped to the bottom, turned to 90 degrees
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Connections:
- net 9*15 renamed 9.42
- net 9*21 renamed 9.29
- net A0 renamed 9.39
- net A1 renamed 9.40
- net A2 renamed 9.37
- net A3 renamed 9.38
- net N$107 renamed 8.17
- net N$109 renamed 9.32
- net N$11 renamed 9.27
- net N$113 renamed 9.30
- net N$115 renamed 8.7
- net N$119 renamed 8.18
- net N$121 renamed 9.12
- net N$124 renamed 9.13
- net N$128 renamed 9.25
- net N$13 renamed 9.41
- net N$131 renamed 9.15
- net N$138 renamed 9.23
- net N$140 renamed 9.17
- net N$141 renamed 9.21
- net N$145 renamed 8.16
- net N$15 renamed 9.26
- net N$2 renamed 8.12
- net N$21 renamed 8.14
- net N$25 renamed 8.13
- net N$27 renamed 8.15
- net N$28 renamed 8.19
- net N$29 renamed 8.26
- net N$3 renamed 9.24
- net N$30 renamed 9.11
- net N$40 renamed 9.19
- net N$41 renamed 8.9
- net N$42 renamed 9.34
- net N$43 renamed 8.8
- net N$44 renamed 8.10
- net N$5 renamed 9.14
- net N$7 renamed 9.16
- net N$9 renamed 9.18
- net N$99 renamed 8.11
Routing:
- net N$147: track 10.8 -> 2.20 mm
- net N$151: track 10.8 -> 2.20 mm
- net N$149: track 10.8 -> 2.20 mm
- net N$146: track 10.8 -> 2.20 mm
- net +3V3: track 101.7 -> 97.4 mm
- net DGND: track 376.9 -> 373.6 mm
- net GND2: track 155.0 -> 152.4 mm
- net XXXXXX: track 135.5 -> 133.1 mm
- net N$136: track 4.52 -> 2.20 mm
- net +5V/2: track 114.9 -> 113.4 mm
- net N$133: track 2.20 -> 3.19 mm
- net N$57: track 35.0 -> 34.0 mm
- net N$50: track 66.0 -> 66.9 mm
- net V-: track 120.7 -> 121.6 mm
- net N$59: track 43.3 -> 42.5 mm
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Other:
- outline, holes or cut-outs redrawn
- board text added: "8.10"
- board text added: "8.16"
- board text added: "8.17"
- board text added: "8.18"
- board text added: "8.7"
- board text added: "8.8"
- board text added: "8.9"
- board text added: "9.11"
- board text added: "9.12"
- board text added: "9.13"
- board text added: "9.15"
- board text added: "9.17"
- board text added: "9.19"
- board text added: "9.21"
- board text added: "9.23"
- board text added: "9.30"
- board text added: "DG1642"
- board text removed: "0.00"
- board text removed: "RX"
- board text removed: "TX"

Commit message: work in progress
Parts:
- removed 9.29, 9.42: TLP2200F, Dean:DIL08-ROUND
- added 0000, 1111: TLP2200F, Dean:DIL08-ROUND
- added C23, C24: (no value), Dean:C0805K
- added C25: (no value), Dean:C0402
- added U$18: LM1117, Dean:SOT223
- C18: device rcl:C0402 -> Dean:C0402
- moved C18 5.63 mm to (36.8, 49.4), turned to 90 degrees
- moved C16 5.39 mm to (38.4, 55.1)
- moved TPS73133 3.73 mm to (38.8, 50.1), turned to 180 degrees
- moved C19 1.91 mm to (4.57, 25.8)
- moved C21 1.60 mm to (45.3, 60.0), turned to 0 degrees
- moved U$5 0.54 mm to (37.7, 41.8)
- moved R14 0.51 mm to (65.7, 38.9)
- moved R15 0.51 mm to (65.7, 49.0)
- moved R16 0.51 mm to (74.9, 37.1)
- moved R38 0.51 mm to (4.19, 19.8)
- moved C14 0.51 mm to (69.3, 40.9)
- moved C15 0.51 mm to (69.3, 51.8)
- moved R17 0.51 mm to (74.7, 48.0)
- moved U$16 0.40 mm to (36.2, 41.8)
Connections:
- net N$80 renamed HSYNC
- net N$81 renamed VSYNC
- net N$82 renamed PCLK
- new net N$2: C23.1, U$18.2, U$18.TAB, U$4.11, U$4.12, U$5.P$1
- net 9.29: now also 1111.2; no longer 9.29.2
- net 9.42: now also 0000.2; no longer 9.42.2
- net DGND: now also C23.2, C24.2, C25.2, U$18.1
- net N$105: now also C24.1, C25.1, U$18.3
- net N$31: now also 0000.3; no longer 9.29.3
- net N$32: now also 1111.3; no longer 9.42.3
- net N$33: now also 0000.5, 0000.6; no longer 9.29.5, 9.29.6
- net N$34: now also 1111.5, 1111.6; no longer 9.42.5, 9.42.6
- net N$45: now also 0000.8; no longer 9.29.8
- net N$46: now also 1111.8; no longer 9.42.8
- net N$47: now also 1111.7; no longer 9.42.7
- net N$48: now also 0000.7; no longer 9.29.7
- net VCC/2: no longer U$4.11, U$4.12, U$5.P$1
Routing:
- net N$105: track 60.8 -> 108.1 mm
- net N$2: track 0.00 -> 35.6 mm
- net 9.29: track 58.7 -> 69.6 mm
- net VCC/2: track 56.1 -> 46.7 mm
- net DGND: track 373.6 -> 381.1 mm, vias 23 -> 26
- net 9.42: track 41.3 -> 34.8 mm
- net HSYNC: track 7.36 -> 11.4 mm, vias 0 -> 1
- net N$69: track 27.4 -> 30.0 mm
- net 8.11: track 34.6 -> 37.1 mm
- net N$130: track 20.2 -> 21.9 mm
- net VSYNC: track 8.67 -> 10.3 mm, vias 0 -> 1
- net PCLK: track 19.8 -> 18.3 mm
- net N$71: track 26.3 -> 24.7 mm, vias 1 -> 0
- net N$68: track 28.1 -> 29.3 mm, vias 1 -> 0
- net N$48: track 14.6 -> 13.6 mm
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- added copper zone on layer 1, net N$2
