File: CNC_IO_Buffer_Cape.sch (EAGLE design)
At the start: 172 parts, among them CN1 1X4-CLEANBIG

Commit message: work in progress
Connections:
- net 9*15 renamed 9.42
- net 9*21 renamed 9.29
- net A0 renamed 9.39
- net A1 renamed 9.40
- net A2 renamed 9.37
- net A3 renamed 9.38
- net N$107 renamed 8.17
- net N$109 renamed 9.32
- net N$11 renamed 9.27
- net N$113 renamed 9.30
- net N$115 renamed 8.7
- net N$119 renamed 8.18
- net N$121 renamed 9.12
- net N$124 renamed 9.13
- net N$128 renamed 9.25
- net N$13 renamed 9.41
- net N$131 renamed 9.15
- net N$138 renamed 9.23
- net N$140 renamed 9.17
- net N$141 renamed 9.21
- net N$145 renamed 8.16
- net N$15 renamed 9.26
- net N$2 renamed 8.12
- net N$21 renamed 8.14
- net N$25 renamed 8.13
- net N$27 renamed 8.15
- net N$28 renamed 8.19
- net N$29 renamed 8.26
- net N$3 renamed 9.24
- net N$30 renamed 9.11
- net N$40 renamed 9.19
- net N$41 renamed 8.9
- net N$42 renamed 9.34
- net N$43 renamed 8.8
- net N$44 renamed 8.10
- net N$5 renamed 9.14
- net N$7 renamed 9.16
- net N$9 renamed 9.18
- net N$99 renamed 8.11
Changed lines of the file:
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@@
 <setting verticaltext="up"/>
 </settings>
-<grid distance="0.05" unitdist="inch" unit="inch" style="lines" multiple="1" display="no" altdistance="0.01" altunitdist="inch" altunit="inch"/>
+<grid distance="0.1" unitdist="inch" unit="inch" style="lines" multiple="1" display="no" altdistance="0.01" altunitdist="inch" altunit="inch"/>
 <layers>
 <layer number="1" name="Top" color="4" fill="1" visible="no" active="no"/>
@@
 </segment>
 </net>
-<net name="N$40" class="0">
+<net name="9.19" class="0">
 <segment>
 <pinref part="U$11" gate="G$1" pin="+"/>
@@
 </segment>
 </net>
-<net name="N$43" class="0">
+<net name="8.8" class="0">
 <segment>
 <pinref part="U$2" gate="G$1" pin="8_GPIO67"/>
@@
 </segment>
 </net>
-<net name="N$44" class="0">
+<net name="8.10" class="0">
 <segment>
 <pinref part="U$2" gate="G$1" pin="10_GPIO68"/>
@@
 </segment>
 </net>
-<net name="N$5" class="0">
+<net name="9.14" class="0">
 <segment>
 <pinref part="U$2" gate="G$1" pin="14_EHRPWM1A"/>
@@
 </segment>
 </net>
-<net name="N$7" class="0">
+<net name="9.16" class="0">
 <segment>
 <pinref part="U$2" gate="G$1" pin="16_EHRPWM1B"/>
@@
 </segment>
 </net>
-<net name="N$9" class="0">
+<net name="9.18" class="0">
 <segment>
 <pinref part="U$2" gate="G$1" pin="18_SPI0_D1"/>
@@
 </segment>
 </net>
-<net name="N$13" class="0">
+<net name="9.41" class="0">
 <segment>
 <pinref part="9.41" gate="G$1" pin="AN"/>
@@
 </segment>
 </net>
-<net name="N$11" class="0">
+<net name="9.27" class="0">
 <segment>
 <pinref part="U$2" gate="G$1" pin="27_GPIO115"/>
@@
 </segment>
 </net>
-<net name="N$3" class="0">
+<net name="9.24" class="0">
 <segment>
 <pinref part="U$2" gate="G$1" pin="24_UART1_TXD"/>
@@
 </segment>
 </net>
-<net name="N$15" class="0">
+<net name="9.26" class="0">
 <segment>
 <pinref part="U$2" gate="G$1" pin="26_UART1_RXD"/>
@@
 </segment>
 </net>
-<net name="N$2" class="0">
+<net name="8.12" class="0">
 <segment>
 <pinref part="U$2" gate="G$1" pin="12_GPIO44"/>
@@
 </segment>
 </net>
-<net name="N$21" class="0">
+<net name="8.14" class="0">
 <segment>
 <pinref part="U$2" gate="G$1" pin="14_GPIO26"/>
@@
 </segment>
 </net>
-<net name="N$25" class="0">
+<net name="8.13" class="0">
 <segment>
 <pinref part="U$2" gate="G$1" pin="13_EHRPWM2B"/>
@@
 </segment>
 </net>
-<net name="N$27" class="0">
+<net name="8.15" class="0">
 <segment>
 <pinref part="U$2" gate="G$1" pin="15_GPIO47"/>
@@
 </segment>
 </net>
-<net name="N$28" class="0">
+<net name="8.19" class="0">
 <segment>
 <pinref part="U$2" gate="G$1" pin="19_EHRPWM2A"/>
@@
 </segment>
 </net>
-<net name="N$29" class="0">
+<net name="8.26" class="0">
 <segment>
 <pinref part="U$2" gate="G$1" pin="26_GPIO61"/>
@@
 </segment>
 </net>
-<net name="N$99" class="0">
+<net name="8.11" class="0">
 <segment>
 <wire x1="256.54" y1="-261.62" x2="297.18" y2="-261.62" width="0.1524" layer="91"/>
@@
 </segment>
 </net>
-<net name="A0" class="0">
+<net name="9.39" class="0">
 <segment>
 <pinref part="U$2" gate="G$1" pin="39_AIN0"/>
@@
 </segment>
 </net>
-<net name="A2" class="0">
+<net name="9.37" class="0">
 <segment>
 <pinref part="U$2" gate="G$1" pin="37_AIN2"/>
@@
 </segment>
 </net>
-<net name="A1" class="0">
+<net name="9.40" class="0">
 <segment>
 <pinref part="U$2" gate="G$1" pin="40_AIN1"/>
@@
 </segment>
 </net>
-<net name="A3" class="0">
+<net name="9.38" class="0">
 <segment>
 <pinref part="U$2" gate="G$1" pin="38_AIN3"/>
@@
 </segment>
 </net>
-<net name="9*15" class="0">
+<net name="9.42" class="0">
 <segment>
 <wire x1="398.78" y1="208.28" x2="581.66" y2="208.28" width="0.1524" layer="91"/>
@@
 </segment>
 </net>
-<net name="9*21" class="0">
+<net name="9.29" class="0">
 <segment>
 <wire x1="302.26" y1="210.82" x2="584.2" y2="210.82" width="0.1524" layer="91"/>
@@
 </segment>
 </net>
-<net name="N$30" class="0">
+<net name="9.11" class="0">
 <segment>
 <pinref part="U$6" gate="G$1" pin="+"/>
@@
 </segment>
 </net>
-<net name="N$115" class="0">
+<net name="8.7" class="0">
 <segment>
 <pinref part="U$12" gate="G$1" pin="+"/>
@@
 </segment>
 </net>
-<net name="N$121" class="0">
+<net name="9.12" class="0">
 <segment>
 <pinref part="U$15" gate="G$1" pin="+"/>
@@
 </segment>
 </net>
-<net name="N$128" class="0">
+<net name="9.25" class="0">
 <segment>
 <pinref part="U$2" gate="G$1" pin="25_GPIO117"/>
@@
 </segment>
 </net>
-<net name="N$124" class="0">
+<net name="9.13" class="0">
 <segment>
 <pinref part="9.3" gate="G$1" pin="AN"/>
@@
 </segment>
 </net>
-<net name="N$131" class="0">
+<net name="9.15" class="0">
 <segment>
 <pinref part="U$1" gate="G$1" pin="+"/>
@@
 </segment>
 </net>
-<net name="N$138" class="0">
+<net name="9.23" class="0">
 <segment>
 <pinref part="U$2" gate="G$1" pin="23_GPIO49"/>
@@
 </segment>
 </net>
-<net name="N$140" class="0">
+<net name="9.17" class="0">
 <segment>
 <pinref part="SPICS3" gate="G$1" pin="A"/>
@@
 </segment>
 </net>
-<net name="N$141" class="0">
+<net name="9.21" class="0">
 <segment>
 <pinref part="U$2" gate="G$1" pin="21_SPI0_DO"/>
@@
 </segment>
 </net>
-<net name="N$41" class="0">
+<net name="8.9" class="0">
 <segment>
 <pinref part="U$13" gate="G$1" pin="+"/>
@@
 </segment>
 </net>
-<net name="N$42" class="0">
+<net name="9.34" class="0">
 <segment>
 <pinref part="U$2" gate="G$1" pin="34_GNDA_ADC"/>
@@
 </segment>
 </net>
-<net name="N$109" class="0">
+<net name="9.32" class="0">
 <segment>
 <pinref part="U$2" gate="G$1" pin="32_VDD_ADC"/>
@@
 </segment>
 </net>
-<net name="N$113" class="0">
+<net name="9.30" class="0">
 <segment>
 <pinref part="U$2" gate="G$1" pin="30_GPIO112"/>
@@
 </segment>
 </net>
-<net name="N$107" class="0">
+<net name="8.17" class="0">
 <segment>
 <pinref part="R22" gate="G$1" pin="1"/>
@@
 </segment>
 </net>
-<net name="N$145" class="0">
+<net name="8.16" class="0">
 <segment>
 <pinref part="R34" gate="G$1" pin="1"/>
@@
 </segment>
 </net>
-<net name="N$119" class="0">
+<net name="8.18" class="0">
 <segment>
 <pinref part="R20" gate="G$1" pin="1"/>

Commit message: work in progress
Parts:
- added C23, C24: (no value), Dean:C-USC0805K
- added C25: (no value), Dean:C-USC0402
- added U$18: LM1117, Dean:LM1117
- C18: device rcl:C-USC0402 -> Dean:C-USC0402
- renumbered 9.29 to 0000, 9.42 to 1111
Connections:
- net N$80 renamed HSYNC
- net N$81 renamed VSYNC
- net N$82 renamed PCLK
- new net N$2: C23.1, U$18.OUT, U$4.11, U$4.12, U$5.1
- net 9.29: now also 1111.AN; no longer 0000.AN
- net 9.42: now also 0000.AN; no longer 1111.AN
- net DGND: now also C23.2, C24.2, C25.2, U$18.GND
- net N$105: now also C24.1, C25.1, U$18.IN
- net VCC/2: no longer U$4.11, U$4.12, U$5.1
Other:
- moved on the sheet: C16, C17, C18, JP22, JP23, JP24, JP25, JP26, JP27, JP28, JP29, JP32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
