File: OPTOCAPE.brd (EAGLE design)
At the start: 79.8 x 80 mm, 176 parts, among them CN1 1X4-CLEANBIG

Commit message: V0.1 Fab version, not yet tested
Parts:
- removed C24: (no value), Dean:C0805K
- C23: value (none) -> 10uf
- moved C25 45.2 mm to (7.24, 12.6), flipped to the bottom
- moved U$16 0.25 mm to (36.2, 41.5)
- moved U$5 0.25 mm to (37.7, 41.5)
- moved C20 0.18 mm to (57.5, 59.6)
- moved C23 0.18 mm to (59.2, 51.2)
- moved C21 0.14 mm to (45.4, 60.1)
Connections:
- net DGND: no longer C24.2
- net N$105: no longer C24.1
Routing:
- net DGND: track 381.1 -> 391.9 mm, vias 26 -> 23
- net N$105: track 108.1 -> 99.4 mm, vias 0 -> 1
- net N$35: track 69.7 -> 68.8 mm
- net N$36: track 57.0 -> 56.3 mm
