File: OPTOCAPE.sch (EAGLE design)
At the start: 176 parts, among them CN1 1X4-CLEANBIG

Commit message: V0.1 Fab version, not yet tested
Parts:
- removed C24: (no value), Dean:C-USC0805K
- C23: value (none) -> 10uf
Connections:
- net DGND: no longer C24.2
- net N$105: no longer C24.1
Other:
- note added: "check shock risk of inverter verify Vout regulation of LM1117 at 0mA"
- note added: "min 10uf"
- moved on the sheet: JP32, JP33, JP34, JP35, JP36, JP37, R20, R21, R22, R23, R34, R35

Commit message: v0.1
Other:
- note removed: "check shock risk of inverter verify Vout regulation of LM1117 at 0mA"
Changed lines of the file:
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@@
 <setting verticaltext="up"/>
 </settings>
-<grid distance="0.05" unitdist="inch" unit="inch" style="lines" multiple="1" display="no" altdistance="0.01" altunitdist="inch" altunit="inch"/>
+<grid distance="0.1" unitdist="inch" unit="inch" style="lines" multiple="1" display="no" altdistance="0.01" altunitdist="inch" altunit="inch"/>
 <layers>
 <layer number="1" name="Top" color="4" fill="1" visible="no" active="no"/>
@@
 <text x="142.24" y="251.46" size="1.778" layer="91">UART4 RX</text>
 <text x="99.06" y="129.54" size="1.778" layer="91">min 10uf</text>
-<text x="360.68" y="-309.88" size="1.778" layer="91">check shock risk of inverter
-verify Vout regulation of LM1117 at 0mA</text>
 </plain>
 <instances>
